File: schematics/src/ioboard/ioboard.brd (EAGLE design)
At the start: 59.1 x 99.1 mm, 39 parts, among them IC1 TL072P

Commit message: Fixed some bugs and updated documentation
Other:
- board text added: "Coron Drum Synth 8 2021 v1.1 GERBSTER.NL"
- board text removed: "Coron Drum Synth 8 2021 GERBSTER.NL"
Changed lines of the file:
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@@
 <wire x1="0" y1="99.05" x2="0" y2="0" width="0" layer="20"/>
 <text x="2.54" y="62.865" size="1.778" layer="25" font="vector">Coron Drum Synth 8
-2021
+2021 v1.1
 GERBSTER.NL</text>
 <hole x="5.08" y="19.05" drill="3.2004"/>
